Commit message: updates

File: Final_Architecture/robots/robot_ver1/CAD/robot_ver1/urdf/robot_ver1.urdf (robot description, URDF)
Before this commit: robot URDF_Files(ver1), 6 links, 5 joints
Links:
- link Base_Link: mass 5.0444 -> 21.810; geometry collision mesh filename=package://robot_ver1/meshes/Base_Link.STL; visual mesh filename=package://robot_ver1/meshes/Base_Link.STL
- link Link_1: mass 3.0503 -> 16.058; geometry collision mesh filename=package://robot_ver1/meshes/Link_1.STL; visual mesh filename=package://robot_ver1/meshes/Link_1.STL
- link Link_2: mass 2.1582 -> 9.843; geometry collision mesh filename=package://robot_ver1/meshes/Link_2.STL; visual mesh filename=package://robot_ver1/meshes/Link_2.STL
- link Link_3: mass 1.1249 -> 7.576; geometry collision mesh filename=package://robot_ver1/meshes/Link_3.STL; visual mesh filename=package://robot_ver1/meshes/Link_3.STL
- link Wrist_1: mass 0.25214 -> 4.535; geometry collision mesh filename=package://robot_ver1/meshes/Wrist_1.STL; visual mesh filename=package://robot_ver1/meshes/Wrist_1.STL
- link Wrist_2: mass 0.25214 -> 4.535; geometry collision mesh filename=package://robot_ver1/meshes/Wrist_2.STL; visual mesh filename=package://robot_ver1/meshes/Wrist_2.STL

Commit message: 6 DOF

File: Final_Architecture/robots/robot_ver1/CAD/robot_ver1/urdf/robot_ver1.urdf (robot description, URDF)
Before this commit: robot robot_ver1, 6 links, 5 joints
Links:
- added link End_Effector, mass 0.183; collision mesh filename=package://robot_ver1/meshes/End_Effector.STL; visual mesh filename=package://robot_ver1/meshes/End_Effector.STL
Joints:
- added joint Joint_6: type revolute, parent Wrist_2, child End_Effector, origin xyz=-0.033 0 -0.1005 rpy=0 1.5708 0, axis 0 0 -1, limit lower=0 upper=0 effort=0 velocity=0

Commit message: robot ver 2 and dynamic analysis

File: Final_Architecture/robots/robot_ver1/CAD/robot_ver1/urdf/robot_ver1.urdf (robot description, URDF)
Before this commit: robot robot_ver1, 7 links, 6 joints
Links:
- link Base_Link: mass 21.810 -> 4.000
- link End_Effector: mass 0.183 -> 0.300
- link Link_1: mass 16.058 -> 2.200
- link Link_2: mass 9.843 -> 3.500
- link Link_3: mass 7.576 -> 2.350
- link Wrist_1: mass 4.535 -> 0.575
- link Wrist_2: mass 4.535 -> 0.575
